Commit message: add set play state and paramters

File: musashi_player_description/robots/musashi_player.urdf.xacro (robot description, xacro)
@@ -2,9 +2,36 @@
 <robot name="musashi" xmlns:xacro="http://ros.org/wiki/xacro">
 <xacro:include filename="$(find musashi_player_description)/urdf/base/base.urdf.xacro"/>
-  <!-- Base -->
+  <!-- base -->
+  <!-- <link name="base_footprint"/>
+  <xacro:base parent="base_footprint"> -->
+	<!-- <origin xyz="0 0 0.028"/> -->
+	<!-- <origin xyz="0 0 0.028"/>
+  </xacro:base> -->
+  <!-- base_footprint Definition -->
   <link name="base_footprint"/>
-  <xacro:base parent="base_footprint">
-	<origin xyz="0 0 0.028"/>
-  </xacro:base>
+  <joint name="base_joint" type="fixed">
+  	<origin xyz="0 0 0.03" rpy="0 0 0"/>
+		<parent link="base_footprint"/>
+		<child link = "base_link"/>
+  </joint>
+	<link name="base_link">
+		<origin xyz="0 0 0" rpy="0 0 0"/>
+		<inertial>
+			<origin xyz="0 0 0"/>
+			<mass value="32"/>
+			<inertia ixx="100" ixy="0" ixz="0" iyy="100" iyz="0" izz="2.86" />
+		</inertial>
+		<visual>
+			<geometry>
+				<mesh filename="package://musashi_player_description/meshes/STL/base/musashi_player_2020_4_27.stl"/>
+			</geometry>
+		</visual>
+		<collision>
+			<geometry>
+				<mesh filename="package://musashi_player_description/meshes/STL/base/musashi_player_2020_4_27.stl"/>
+			</geometry>
+		</collision>
+	</link>
+  <!-- gazebo -->
   <gazebo>
     <plugin name="player_controller" filename="libgazebo_ros_planar_move.so">
@@ -16,3 +43,4 @@
     </plugin>
   </gazebo>
+	<!-- end base -->
 </robot>

File: musashi_player_description/urdf/base/base.urdf.xacro (robot description, xacro)
@@ -1,5 +1,7 @@
 <?xml version="1.0"?>
 <robot xmlns:xacro="http://ros.org/wiki/xacro">
+<!-- not use
   <xacro:include filename="$(find musashi_player_description)/urdf/base/base.gazebo.xacro"/>
+-->
 	<xacro:macro name="base" params="parent *joint_origin">
 		<joint name="base_link_joint" type="fixed">
@@ -7,14 +9,15 @@
 			<parent link="${parent}"/>
 			<child link="base_link"/>
+			<dynamics damping="0.1"/>
 		</joint>
 		<link name="base_link">
 			<visual>
 				<geometry>
-					<mesh filename="package://musashi_player_description/meshes/DAE/base/base_link.dae"/>
+					<mesh filename="package://musashi_player_description/meshes/DAE/base/musashi_player_2020_4_27.dae"/>
 				</geometry>
 			</visual>
 			<collision>
 				<geometry>
-					<mesh filename="package://musashi_player_description/meshes/STL/base/base_link.stl"/>
+					<mesh filename="package://musashi_player_description/meshes/STL/base/musashi_player_2020_4_27.stl"/>
 				</geometry>
 			</collision>
